File: PI-Outline.brd (EAGLE design)
At the start: 65 x 30 mm, 15 parts, among them J1 CONNECTOR_PI_40_PIN, J2 Barrel DC In, J3 OLED, J4 VE.Direct Serial, J5 External DS18B20 Temp, J6 FTDI Serial Console, J7 MagJack, U1 OLED_I2C, U2 SI7006-A20-IM, U3 HAT EEPROM, U4 INA260AIPW, U5 Isolator, U6 ENC28J60_SS, U7 5V SMPS, Y1 ECS-250-20-3X-EN-TR

Commit message: README
Parts:
- removed J3: OLED, APU_ENGR480_UPS_EAGLE_Library:ESQ-104-XX-X-S
- removed U1: OLED_I2C, APU_ENGR480_UPS_EAGLE_Library:OLED-I2C
- moved J1 31.6 mm to (3.50, 39.0)
- moved U3 31.1 mm to (29.0, -21.0)
- moved U4 23.0 mm to (-10.5, -28.0)
Connections:
- removed net MISO: J1.21, U6.6
- removed net MOSI: J1.19, U6.7
- removed net N$1: J1.8, J6.4
- removed net N$2: J1.10, J6.5
- removed net N$4: J1.7, J5.2
- removed net SCK: J1.5, J3.3, U2.6, U4.9
- removed net SCLK: J1.23, U6.8
- removed net SDA: J1.3, J3.4, U2.1, U4.8
- new net S$1: J5.1, J6.1, J7.S1, J7.S2, U2.2, U6.18, U6.2, U6.21, U6.22
- new net S$2: U4.11, U4.4, U4.6
- new net S$3: U2.1, U4.8
- new net S$5: U2.6, U4.9
- net 3.3V: no longer J1.1, J3.2
- net GND: no longer J3.1, J5.1, J6.1, J7.S1, J7.S2, U2.2, U4.11, U4.4, U4.6, U6.18, U6.2, U6.21, U6.22, U7.2
