File: UPS-MAF-APU.brd (EAGLE design)
At the start: 65 x 30 mm, 15 parts, among them J1 CONNECTOR_PI_40_PIN, J2 Barrel DC In, J3 OLED, J4 VE.Direct Serial, J5 External DS18B20 Temp, J6 FTDI Serial Console, J7 MagJack, U1 OLED_I2C, U2 SI7006-A20-IM, U3 HAT EEPROM, U4 INA260AIPW, U5 Isolator, U6 ENC28J60_SS, U7 5V SMPS, Y1 ECS-250-20-3X-EN-TR

Commit message: README
Parts:
- removed U3: HAT EEPROM, APU_ENGR480_UPS_EAGLE_Library:SOP65P640X120-8N
- removed U5: Isolator, APU_ENGR480_UPS_EAGLE_Library:SOIC127P600X175-8N
- added C1: 10nF, resistor:C0603
- added C2, C3, C5, C6, C7, C9: 100nF, resistor:C0603
- added C4: 10uF, resistor:C0603
- added C8: 18pF, resistor:C0603
- added FB!: 600 uH, adafruit:R0805
- added R1, R2: 180, SparkFun-Resistors:0603
- added R3, R4, R5, R6, R9: 49.9, adafruit:R0805
- added R7: 100K, adafruit:R0805
- added R8: 2.2K, SparkFun-Resistors:0603
- J4: value VE.Direct Serial -> OSTOQ045451; device APU_ENGR480_UPS_EAGLE_Library:S4B-PH-SM4-TB -> APU_ENGR480_UPS_EAGLE_Library:OSTOQ045451
- Y1: device ECS-250-20-3X-EN-TR:ECS250203XENTR -> APU_ENGR480_UPS_EAGLE_Library:ECS250203XENTR
- moved Y1 176.2 mm to (-35.6, 88.9)
- moved J6 112.0 mm to (-30.5, 59.7)
- moved U2 109.0 mm to (-53.3, 94.0)
- moved J7 98.0 mm to (-22.9, 11.4)
- moved J3 95.9 mm to (-19.1, 81.3), turned to 0 degrees
- moved U4 93.1 mm to (-31.8, 80.0)
- moved J1 84.6 mm to (-39.4, 71.1)
- moved U6 80.9 mm to (-59.7, 45.7)
- moved J4 77.1 mm to (-33.0, 36.8)
- moved U1 72.9 mm to (-33.0, 47.0), turned to 0 degrees
- moved J5 32.7 mm to (-61.0, 7.62)
- moved U7 28.7 mm to (-38.1, 8.89)
- moved J2 24.2 mm to (-53.3, 6.35)
Connections:
- removed net VDDTX: U6.15
- removed net VSSRX: U6.11
- new net 5V: J1.2, J1.4, J6.3, U7.3
- new net INT: J1.22, U6.4
- new net LEDA: J7.L3, U6.27
- new net LEDB: J7.L1, U6.26
- new net N$10: J1.1, J5.3, U2.5
- new net N$9: R8.2, U6.14
- new net OIN: C9.1, R9.1, Y1.1
- new net OOUT: C8.1, U6.23, Y1.2
- new net RST: R7.2, U6.10
- new net RX_OT: J1.10, J6.4
- new net TPIN+: J7.R7, R4.2, U6.13
- new net TPIN-: J7.R8, R3.2, U6.12
- new net TPOUT+: J7.R1, R6.2, U6.17
- new net TPOUT-: J7.R2, R5.2, U6.16
- new net TX_OR: J1.8, J6.5
- new net VIN: J2.1, U7.1
- net 3.3V: now also C2.1, FB!.1, FB!.2, J1.17, J7.R3, R5.1, R6.1; no longer J1.1, J5.3, J6.3, U6.19, U6.20, U6.28
- net BATTERY+: now also J4.1
- net BATTERY-: now also J4.4
- net CS: now also U6.9
- net GND: now also C1.2, C2.2, C3.2, C4.2, C5.2, C6.2, C7.2, C8.2, C9.2, J1.20, J1.9, J2.2, J4.2, J4.3, R1.1, R2.1, R7.1, R8.1, U6.11
- net N$1: now also C1.1, R3.1, R4.1; no longer J1.8, J6.4
- net N$2: now also R9.2, U6.24; no longer J1.10, J6.5
- net N$3: now also C4.1, U6.1; no longer U6.13
- net N$5: now also J7.L2, R2.2; no longer U6.12
- net N$6: now also U6.3; no longer J7.R2, U6.16
- net N$7: now also J7.L4, R1.2; no longer J7.R1, U6.17
- net VDD: now also C3.1, C5.1, C6.1, C7.1, U6.15, U6.19, U6.20, U6.28; no longer U2.5
Other:
- board size 65 x 30 mm -> 160 x 100 mm
- board text removed: "APU MAF UPS 2019 2/25/19"
- board text removed: "Bottom"
- board text removed: "Top"

Commit message: README
Changed lines of the file:
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@@
 <attribute name="MF" value="WIZnet" x="0" y="0" size="1.778" layer="27" display="off"/>
 <attribute name="MP" value="RB1-125BAG1A" x="0" y="0" size="1.778" layer="27" display="off"/>
+<attribute name="NAME" x="-22.86" y="11.43" size="5.08" layer="51" align="center"/>
 <attribute name="NAME" x="-22.860790625" y="23.939" size="1.778" layer="25" font="vector" align="center"/>
-<attribute name="NAME" x="-22.86" y="11.43" size="5.08" layer="51" align="center"/>
 <attribute name="PACKAGE" value="None" x="0" y="0" size="1.778" layer="27" display="off"/>
 <attribute name="PRICE" value="2.18 USD" x="0" y="0" size="1.778" layer="27" display="off"/>

Commit message: deleted and re-created .brd file to get them back in sync.
 Please enter the commit message for your changes. Lines starting
Parts:
- R7: value 100K -> 10K
- R9: value 49.9 -> 0
- moved C7 56.2 mm to (-73.7, 88.9)
- moved R6 52.8 mm to (-68.6, 80.0)
- moved R7 24.1 mm to (-73.7, 80.0)
- moved C3 7.62 mm to (-50.8, 88.9)
- moved C5 7.62 mm to (-58.4, 88.9)
- moved C8 7.62 mm to (-36.8, 95.2)
- moved R2 7.62 mm to (-58.4, 94.0)
- moved U2 7.62 mm to (-45.7, 94.0)
- moved C1 7.62 mm to (-24.1, 95.2)
- moved C4 7.62 mm to (-30.5, 95.2)
- moved Y1 7.62 mm to (-27.9, 88.9)
- moved R9 7.62 mm to (-15.2, 88.9)
- moved C2 7.62 mm to (-43.2, 88.9)
- moved C9 7.62 mm to (-17.8, 95.2)
- moved R1 7.62 mm to (-54.6, 94.0)
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Connections:
- removed net VDD: C3.1, C5.1, C6.1, C7.1, U6.15, U6.19, U6.20, U6.28
- net 3.3V: now also C3.1, C5.1, C6.1, C7.1, U4.6, U6.15, U6.19, U6.20, U6.28
- net GND: no longer U4.6

Commit message: README
Other:
- board size 160 x 100 mm -> 65 x 30 mm
- board text added: "APU MAF UPS 2019 2/25/19"
Changed lines of the file:
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@@
 <?xml version="1.0" encoding="utf-8"?>
 <!DOCTYPE eagle SYSTEM "eagle.dtd">
-<eagle version="9.3.1">
+<eagle version="9.3.0">
 <drawing>
 <settings>
@@
 <board>
 <plain>
-<wire x1="0" y1="0" x2="160" y2="0" width="0" layer="20"/>
-<wire x1="160" y1="0" x2="160" y2="100" width="0" layer="20"/>
-<wire x1="160" y1="100" x2="0" y2="100" width="0" layer="20"/>
-<wire x1="0" y1="100" x2="0" y2="0" width="0" layer="20"/>
+<hole x="54.8" y="47.43" drill="2.75"/>
+<wire x1="51.3" y1="47.43" x2="54.8" y2="43.93" width="0" layer="20" curve="90"/>
+<hole x="112.8" y="47.43" drill="2.75"/>
+<wire x1="112.8" y1="43.93" x2="116.3" y2="47.43" width="0" layer="20" curve="90"/>
+<hole x="112.8" y="70.43" drill="2.75"/>
+<wire x1="116.3" y1="70.43" x2="112.8" y2="73.93" width="0" layer="20" curve="90"/>
+<hole x="54.8" y="70.43" drill="2.75"/>
+<wire x1="54.8" y1="73.93" x2="51.3" y2="70.43" width="0" layer="20" curve="90"/>
+<wire x1="51.3" y1="47.43" x2="51.3" y2="70.43" width="0" layer="20"/>
+<wire x1="54.8" y1="73.93" x2="112.8" y2="73.93" width="0" layer="20"/>
+<wire x1="116.3" y1="70.43" x2="116.3" y2="47.43" width="0" layer="20"/>
+<wire x1="54.8" y1="43.93" x2="112.8" y2="43.93" width="0" layer="20"/>
+<circle x="54.8" y="47.43" radius="3.1" width="0" layer="41"/>
+<circle x="54.8" y="47.43" radius="3.1" width="0" layer="29"/>
+<circle x="54.8" y="47.43" radius="3.1" width="0" layer="40"/>
+<circle x="54.8" y="47.43" radius="3.1" width="0" layer="30"/>
+<circle x="54.8" y="70.43" radius="3.1" width="0" layer="41"/>
+<circle x="54.8" y="70.43" radius="3.1" width="0" layer="29"/>
+<circle x="54.8" y="70.43" radius="3.1" width="0" layer="40"/>
+<circle x="54.8" y="70.43" radius="3.1" width="0" layer="30"/>
+<circle x="112.8" y="70.43" radius="3.1" width="0" layer="41"/>
+<circle x="112.8" y="70.43" radius="3.1" width="0" layer="29"/>
+<circle x="112.8" y="70.43" radius="3.1" width="0" layer="40"/>
+<circle x="112.8" y="70.43" radius="3.1" width="0" layer="30"/>
+<circle x="112.8" y="47.43" radius="3.1" width="0" layer="41"/>
+<circle x="112.8" y="47.43" radius="3.1" width="0" layer="29"/>
+<circle x="112.8" y="47.43" radius="3.1" width="0" layer="40"/>
+<circle x="112.8" y="47.43" radius="3.1" width="0" layer="30"/>
+<text x="102.8" y="44.43" size="3" layer="22" font="vector" rot="MR0">APU MAF UPS 2019
+2/25/19</text>
 </plain>
 <attributes>
@@
 <attribute name="MF" value="WIZnet" x="0" y="0" size="1.778" layer="27" display="off"/>
 <attribute name="MP" value="RB1-125BAG1A" x="0" y="0" size="1.778" layer="27" display="off"/>
+<attribute name="NAME" x="-22.86" y="11.43" size="5.08" layer="51" align="center"/>
 <attribute name="NAME" x="-22.860790625" y="23.939" size="1.778" layer="25" font="vector" align="center"/>
-<attribute name="NAME" x="-22.86" y="11.43" size="5.08" layer="51" align="center"/>
 <attribute name="PACKAGE" value="None" x="0" y="0" size="1.778" layer="27" display="off"/>
 <attribute name="PRICE" value="2.18 USD" x="0" y="0" size="1.778" layer="27" display="off"/>
@@
 </drawing>
 <compatibility>
+<note version="6.3" minversion="6.2.2" severity="warning">
+Since Version 6.2.2 text objects can contain more than one line,
+which will not be processed correctly with this version.
+</note>
 <note version="8.2" severity="warning">
 Since Version 8.2, EAGLE supports online libraries. The ids
