File: UPS-MAF-APU.brd (EAGLE design)
At the start: 160 x 100 mm, 32 parts, among them J1 CONNECTOR_PI_40_PIN, J2 Barrel DC In, J3 OLED, J4 OSTOQ045451, J5 External DS18B20 Temp, J6 FTDI Serial Console, J7 MagJack, U1 OLED_I2C, U2 SI7006-A20-IM, U4 INA260AIPW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

Commit message: README
Parts:
- moved J1 126.0 mm to (86.4, 62.2)
Connections:
- net 3.3V: no longer U4.6
- net GND: now also U4.6
Other:
- board size 160 x 100 mm -> 65 x 30 mm
- board text added: "APU MAF UPS 2019 2/25/19"
- board text added: "Bottom"
- board text added: "TOP"

Commit message: README
Parts:
- moved J1 38.8 mm to (53.3, 82.5)
Connections:
- removed net N$6 (its old number): U6.3
- new net N$2: R10.2, Y1.2
- net INT: now also U6.4
- net OOUT: no longer R10.2, Y1.2
Other:
- board size 65 x 30 mm -> 65 x 56 mm

Commit message: README
Parts:
- moved J4 51.7 mm to (12.5, 12.3)
- moved J1 36.6 mm to (32.5, 52.5)

Commit message: README
Parts:
- moved R9 130.3 mm to (59.9, 13.5)
- moved C9 129.1 mm to (60.2, 25.2)
- moved R10 118.9 mm to (59.6, 8.40)
- moved J5 111.6 mm to (49.6, 22.5), turned to 270 degrees
- moved R4 111.2 mm to (29.1, 34.5)
- moved C8 110.7 mm to (8.39, 4.25)
- moved C2 107.1 mm to (15.4, 22.4)
- moved J6 105.5 mm to (62.9, 10.5), turned to 90 degrees
- moved R3 103.4 mm to (28.5, 38.0)
- moved R1 103.4 mm to (18.6, 45.0)
- moved C1 101.7 mm to (30.0, 43.4)
- moved FB! 99.5 mm to (17.3, 17.0)
- moved U6 98.7 mm to (38.7, 38.7)
- moved U2 97.5 mm to (17.0, 39.0), turned to 270 degrees
- moved R6 91.0 mm to (12.1, 4.90)
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Routing:
- added copper zone on layer 16, net GND

Commit message: README
Parts:
- moved R6 42.8 mm to (38.0, 39.0), turned to 180 degrees
- moved R10 39.1 mm to (52.6, 46.9)
- moved R9 36.8 mm to (27.0, 30.0)
- moved FB! 35.6 mm to (38.0, 46.0)
- moved C9 26.4 mm to (35.0, 33.0)
- moved C2 26.4 mm to (38.0, 36.0), turned to 180 degrees
- moved R1 23.6 mm to (42.0, 48.0)
- moved C3 22.4 mm to (33.5, 43.5)
- moved R7 22.3 mm to (17.5, 23.0), turned to 180 degrees
- moved C6 18.4 mm to (33.5, 48.5)
- moved C7 18.1 mm to (33.5, 46.0)
- moved C8 16.5 mm to (17.5, 18.0)
- moved C1 15.3 mm to (15.0, 40.5), turned to 90 degrees
- moved U6 12.9 mm to (27.0, 44.0)
- moved R5 12.8 mm to (38.0, 42.5), turned to 180 degrees
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Routing:
- net GND: track 0.00 -> 312.3 mm
- net 3.3V: track 0.00 -> 216.0 mm, vias 0 -> 3
- net 5V: track 0.00 -> 118.1 mm
- net N$4: track 0.00 -> 90.2 mm
- net RX_OT: track 0.00 -> 83.2 mm, vias 0 -> 1
- net SCK: track 0.00 -> 82.1 mm, vias 0 -> 2
- net TX_OR: track 0.00 -> 71.1 mm, vias 0 -> 1
- net SDA: track 0.00 -> 67.2 mm
- net OOUT: track 0.00 -> 66.0 mm, vias 0 -> 3
- net N$2: track 0.00 -> 47.2 mm, vias 0 -> 2
- net LEDB: track 0.00 -> 46.9 mm, vias 0 -> 1
- net LEDA: track 0.00 -> 44.7 mm, vias 0 -> 2
- net VIN: track 0.00 -> 40.7 mm, vias 0 -> 1
- net N$7: track 0.00 -> 36.7 mm
- net OIN: track 0.00 -> 36.6 mm, vias 0 -> 3
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Other:
- board text added: "APU MAF UPS 2019 4/7/2019"
- board text removed: "APU MAF UPS 2019 2/25/19"

Commit message: README
Parts:
- removed FB!: 600 uH, adafruit:R0805
- added FB1: 600 uH, adafruit:R0805
- added R11: 0, adafruit:R0805
- added R12, R8: 4.7K, adafruit:R0805
- C9: value 100nF -> 18pF
- R10: value 0 -> 4.7K
- moved R10 48.2 mm to (8.00, 28.5), turned to 90 degrees
- moved R7 31.1 mm to (36.0, 48.0)
- moved C1 27.5 mm to (42.5, 40.5), flipped to the bottom, turned to 270 degrees
- moved J6 27.2 mm to (36.0, 6.00), flipped to the bottom, turned to 180 degrees
- moved R1 26.5 mm to (61.5, 30.0)
- moved R3 26.3 mm to (45.0, 47.0), flipped to the bottom, turned to 270 degrees
- moved R4 26.3 mm to (45.0, 42.5), flipped to the bottom, turned to 90 degrees
- moved R9 22.5 mm to (40.5, 48.0)
- moved C4 22.2 mm to (30.5, 47.5), flipped to the bottom, turned to 180 degrees
- moved U7 19.7 mm to (20.0, 32.0), flipped to the top
- moved U2 18.0 mm to (9.50, 33.5)
- moved J4 17.0 mm to (3.50, 29.5), turned to 270 degrees
- moved C8 16.5 mm to (34.0, 18.5)
- moved Y1 16.0 mm to (34.0, 25.5)
- moved R2 15.5 mm to (61.5, 48.0)
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Connections:
- net TPIN+ renamed TPIN_P
- net TPIN- renamed TPIN_N
- net TPOUT+ renamed TPOUT_P
- net TPOUT- renamed TPOUT_N
- new net N$1: C2.1, FB1.2, J7.R3, R5.1, R6.1
- net 3.3V: now also FB1.1, R10.1, R12.1, R8.1; no longer C2.1, FB!.1, FB!.2, J7.R3, R5.1, R6.1
- net N$2: now also C8.1, R11.1; no longer R10.2
- net N$4: now also R8.2
- net OOUT: now also R11.2; no longer C8.1, R10.1
- net SCK: now also R10.2
- net SDA: now also R12.2
Routing:
- net GND: track 312.3 -> 83.0 mm, vias 0 -> 1
- net 5V: track 118.1 -> 67.5 mm, vias 0 -> 1
- net OOUT: track 66.0 -> 15.8 mm, vias 3 -> 1
- net N$2: track 47.2 -> 8.81 mm, vias 2 -> 0
- net 3.3V: track 216.0 -> 179.7 mm, vias 3 -> 2
- net N$4: track 90.2 -> 55.7 mm
- net N$7: track 36.7 -> 2.91 mm
- net RX_OT: track 83.2 -> 58.2 mm, vias 1 -> 0
- net OIN: track 36.6 -> 13.3 mm, vias 3 -> 1
- net RST: track 27.4 -> 4.18 mm, vias 0 -> 1
- net N$1: track 0.00 -> 21.7 mm
- net CS: track 29.5 -> 9.50 mm, vias 2 -> 0
- net VIN: track 40.7 -> 22.2 mm, vias 1 -> 0
- net BATTERY+: track 32.6 -> 14.3 mm
- net SCLK: track 24.4 -> 6.39 mm, vias 2 -> 0
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
Commit message: README
Routing:
- net N$8: track 0.00 -> 21.3 mm, vias 0 -> 3
- net OIN: track 13.3 -> 13.9 mm
Changed lines of the file:
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@@
 <attribute name="MF" value="WIZnet" x="69.43" y="61.86" size="1.778" layer="27" rot="R90" display="off"/>
 <attribute name="MP" value="RB1-125BAG1A" x="69.43" y="61.86" size="1.778" layer="27" rot="R90" display="off"/>
+<attribute name="NAME" x="58" y="39" size="5.08" layer="51" rot="R90" align="center"/>
 <attribute name="NAME" x="45.491" y="38.999209375" size="1.778" layer="25" font="vector" rot="R90" align="center"/>
-<attribute name="NAME" x="58" y="39" size="5.08" layer="51" rot="R90" align="center"/>
 <attribute name="PACKAGE" value="None" x="69.43" y="61.86" size="1.778" layer="27" rot="R90" display="off"/>
 <attribute name="PRICE" value="2.18 USD" x="69.43" y="61.86" size="1.778" layer="27" rot="R90" display="off"/>
@@
 <wire x1="12.275" y1="18.562" x2="11.625" y2="18.562" width="0" layer="19" extent="1-1"/>
 </signal>
-<signal name="UPSIN">
+<signal name="UPSIN" class="1">
 <contactref element="U4" pad="1"/>
 <contactref element="U4" pad="3"/>
@@
 <wire x1="33.2232" y1="32.004" x2="33.15" y2="32" width="0.1524" layer="1"/>
 <via x="33.909" y="39.3954" extent="1-16" drill="0.35"/>
+<wire x1="33.909" y1="39.3954" x2="34.0136" y2="39.5" width="0.1524" layer="16"/>
+<wire x1="34.0136" y1="39.5" x2="34.5" y2="39.5" width="0.1524" layer="16"/>
 </signal>
 <signal name="OOUT">
@@
 <wire x1="48.28534375" y1="33.5" x2="45" y2="33.5" width="0.2032" layer="16"/>
 </signal>
+<signal name="N$8">
+<via x="37" y="39.5" extent="1-16" drill="0.35"/>
+<wire x1="37" y1="39.5" x2="37" y2="41.5" width="0.1524" layer="1"/>
+<wire x1="37" y1="41.5" x2="32.5" y2="41.5" width="0.1524" layer="1"/>
+<via x="32.5" y="41.5" extent="1-16" drill="0.35"/>
+<wire x1="32.5" y1="41.5" x2="32.5" y2="42" width="0.1524" layer="16"/>
+<wire x1="32.5" y1="41.5" x2="31.5" y2="41.5" width="0.1524" layer="16"/>
+<wire x1="32.5" y1="41.5" x2="32.5" y2="43" width="0.1524" layer="16"/>
+<wire x1="32.5" y1="41.5" x2="33.5" y2="41.5" width="0.1524" layer="16"/>
+<wire x1="32.5" y1="41.5" x2="32.5" y2="40.5" width="0.1524" layer="16"/>
+<wire x1="37" y1="39.5" x2="37.5" y2="39.5" width="0.1524" layer="16"/>
+<wire x1="37" y1="41.5" x2="39" y2="39.5" width="0.1524" layer="1"/>
+<wire x1="39" y1="39.5" x2="45.5" y2="39.5" width="0.1524" layer="1"/>
+<via x="45.5" y="39.5" extent="1-16" drill="0.35"/>
+</signal>
 </signals>

Commit message: README
Parts:
- moved J5 52.5 mm to (14.0, 1.00), turned to 0 degrees
- moved R10 49.2 mm to (54.5, 12.5), turned to 180 degrees
- moved R8 46.0 mm to (8.00, 12.0)
- moved J4 43.7 mm to (37.5, 2.00), turned to 0 degrees
- moved J6 43.0 mm to (2.50, 33.0), flipped to the top, turned to 90 degrees
- moved U2 40.6 mm to (44.5, 13.0), flipped to the bottom, turned to 180 degrees
- moved J2 39.6 mm to (30.5, 5.65), turned to 180 degrees
- moved U4 38.0 mm to (45.5, 8.00), turned to 0 degrees
- moved J3 33.5 mm to (49.2, 19.2), turned to 270 degrees
- moved R12 22.5 mm to (36.5, 11.5)
- moved C8 19.5 mm to (21.5, 33.5), flipped to the bottom
- moved R11 13.6 mm to (28.0, 37.5), flipped to the bottom, turned to 180 degrees
- moved U1 13.3 mm to (31.5, 19.2), turned to 180 degrees
- moved Y1 9.71 mm to (28.5, 33.5), flipped to the bottom, turned to 0 degrees
- moved U7 6.95 mm to (14.0, 35.5), flipped to the bottom
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Routing:
- net TX_OR: track 63.5 -> 19.5 mm
- net 3.3V: track 179.7 -> 221.5 mm, vias 2 -> 1
- net GND: track 83.0 -> 43.2 mm, vias 1 -> 0
- net SDA: track 51.4 -> 86.6 mm
- net RX_OT: track 58.2 -> 27.4 mm
- net 5V: track 67.5 -> 37.4 mm, vias 1 -> 0
- net N$8: track 21.3 -> 0.00 mm, vias 3 -> 0
- net N$6: track 10.8 -> 22.5 mm, vias 2 -> 0
- net TPOUT_P: track 28.4 -> 19.2 mm
- net OOUT: track 15.8 -> 7.41 mm, vias 1 -> 0
- net N$4: track 55.7 -> 49.2 mm
- net OIN: track 13.9 -> 7.53 mm, vias 1 -> 0
- net N$1: track 21.7 -> 27.7 mm
- net N$7: track 2.91 -> 8.83 mm
- net SCK: track 73.5 -> 78.8 mm, vias 0 -> 1
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