File: UPS-MAF-APU.brd (EAGLE design)
At the start: 65 x 56 mm, 35 parts, among them J1 CONNECTOR_PI_40_PIN, J2 Barrel DC In, J3 OLED, J4 OSTOQ045451, J5 External DS18B20 Temp, J6 FTDI Serial Console, J7 MagJack, U1 OLED_I2C, U2 SI7006-A20-IM, U4 INA260AIPW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

Commit message: README
Parts:
- removed R11: 0, adafruit:R0805
- moved C8 15.7 mm to (35.8, 27.0), turned to 180 degrees
- moved R2 14.7 mm to (46.8, 47.0), turned to 90 degrees
- moved U2 11.2 mm to (38.5, 22.5), turned to 90 degrees
- moved R10 10.5 mm to (54.5, 23.0)
- moved J3 9.85 mm to (45.2, 28.2)
- moved U1 9.85 mm to (27.5, 28.2)
- moved U4 9.55 mm to (44.5, 17.5)
- moved C9 9.10 mm to (32.8, 27.0), turned to 0 degrees
- moved C7 9.01 mm to (31.0, 35.0)
- moved J4 9.01 mm to (37.0, 11.0)
- moved C6 8.31 mm to (38.2, 34.5)
- moved C5 7.00 mm to (40.8, 34.5)
- moved R12 6.96 mm to (34.0, 18.0)
- moved R8 6.50 mm to (5.50, 18.0)
- moved Y1 6.49 mm to (34.2, 30.5), turned to 180 degrees
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Connections:
- removed net N$2: C8.1, R11.1, Y1.2
- net OOUT: now also C8.1, Y1.2; no longer R11.2
Routing:
- net LEDA: track 31.9 -> 74.4 mm, vias 1 -> 0
- net 3.3V: track 221.5 -> 179.4 mm, vias 1 -> 4
- net LEDB: track 33.7 -> 64.0 mm, vias 1 -> 0
- net GND: track 43.2 -> 69.2 mm, vias 0 -> 1
- net N$5: track 5.44 -> 18.1 mm
- net BATTERY+: track 16.7 -> 27.5 mm
- net RX_OT: track 27.4 -> 17.0 mm
- net N$2: track 7.99 -> 0.00 mm
- net OOUT: track 7.41 -> 14.2 mm
- net N$6: track 22.5 -> 29.1 mm
- net OIN: track 7.53 -> 14.1 mm
- net TX_OR: track 19.5 -> 13.4 mm
- net SDA: track 86.6 -> 80.8 mm, vias 0 -> 2
- net VIN: track 26.0 -> 21.5 mm
- net 5V: track 37.4 -> 34.0 mm
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