File: UPS-MAF-APU.sch (EAGLE design)
At the start: 32 parts, among them J1 CONNECTOR_PI_40_PIN, J2 Barrel DC In, J3 OLED, J4 OSTOQ045451, J5 External DS18B20 Temp, J6 FTDI Serial Console, J7 MagJack, U1 OLED_I2C, U2 SI7006-A20-IM, U4 INA260AIPW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

Commit message: README
Parts:
- R7: value 100K -> 10K
- R9: value 49.9 -> 0
Connections:
- removed net VDD: C3.1, C5.1, C6.1, C7.1, U6.VDD, U6.VDDPLL, U6.VDDRX, U6.VDDTX
- net 3.3V: now also C3.1, C5.1, C6.1, C7.1, U4.GND_1, U6.VDD, U6.VDDPLL, U6.VDDRX, U6.VDDTX
- net GND: now also U2.GND; no longer U4.GND_1
Other:
- note added: "I2C Address 0x41"
- note removed: "add battery/charger connector add power, status lights"
- moved on the sheet: C1, C2, C3, C5, C6, C7, R2, R9, U1

Commit message: README
Parts:
- removed R8: 2.2K, SparkFun-Resistors:180OHM-0603-1/10W-1%
- added R10: 0, adafruit:R-US_R0805
- C1: value 10nF -> 100nF
- C4: device resistor:C-USC0603 -> resistor:C-USC0805
- R3: value 49.9 -> 50 1%; CRCW060350R0FKEA (none) -> 50
- R4, R5, R6: value 49.9 -> 50 1%
- R9: value 0 -> 2.32K 1%
Connections:
- removed net BATTERY-: J4.4, U4.IN+_1, U4.IN+_2, U4.IN+_3
- removed net N$10: J1.3.3V@1, J5.3, U2.VDD
- removed net N$2: R9.2, U6.OSC2
- new net UPSIN: J4.1, U4.IN+_1, U4.IN+_2, U4.IN+_3
- net 3.3V: now also J1.3.3V@1, J5.3, R7.1, U2.VDD
- net BATTERY+: now also J4.4; no longer J4.1
- net GND: now also R9.2; no longer R7.1, R8.1
- net INT: no longer U6.!INT
- net N$9: now also R9.1; no longer R8.2
- net OIN: now also U6.OSC2; no longer R9.1
- net OOUT: now also R10.1, R10.2
Other:
- note added: "I2C Address 0x40"
- note removed: "I2C Address 0x??"
- moved on the sheet: C8, J4, R7, R9

Commit message: README
Connections:
- net 3.3V: no longer U4.GND_1
- net GND: now also U4.GND_1
Changed lines of the file:
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@@
 <label x="35.56" y="193.04" size="1.778" layer="95"/>
+</segment>
+<segment>
+<pinref part="U4" gate="G$1" pin="GND_1"/>
+<wire x1="33.02" y1="160.02" x2="30.48" y2="160.02" width="0.1524" layer="91"/>
+<label x="27.94" y="160.02" size="1.778" layer="95"/>
 </segment>
 </net>
@@
 </segment>
 <segment>
-<pinref part="U4" gate="G$1" pin="GND_1"/>
-<wire x1="33.02" y1="160.02" x2="30.48" y2="160.02" width="0.1524" layer="91"/>
-<label x="27.94" y="160.02" size="1.778" layer="95"/>
-</segment>
-<segment>

Commit message: README
Connections:
- removed net N$6 (its old number): U6.CLKOUT
- new net N$2: R10.2, Y1.OUT/IN
- net INT: now also U6.!INT
- net OOUT: no longer R10.2, Y1.OUT/IN
Changed lines of the file:
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@@
 <text x="27.94" y="129.54" size="1.778" layer="91" rot="R180" align="top-right">N/C</text>
 <text x="33.02" y="157.48" size="1.778" layer="91" rot="R180" align="top-left">N/C</text>
-<text x="27.94" y="132.08" size="1.778" layer="91" rot="R180" align="top-right">N/C</text>
+<text x="27.94" y="134.62" size="1.778" layer="91" rot="R180" align="top-right">N/C</text>
 </plain>
 <instances>
@@
 </segment>
 </net>
-<net name="N$6" class="0">
-<segment>
-<pinref part="U6" gate="G$1" pin="CLKOUT"/>
-<wire x1="33.02" y1="134.62" x2="20.32" y2="134.62" width="0.1524" layer="91"/>
-</segment>
-</net>
 <net name="INT" class="0">
 <segment>
@@
 <wire x1="175.26" y1="119.38" x2="180.34" y2="119.38" width="0.1524" layer="91"/>
 <label x="180.34" y="119.38" size="1.778" layer="95"/>
+</segment>
+<segment>
+<pinref part="U6" gate="G$1" pin="!INT"/>
+<wire x1="33.02" y1="132.08" x2="27.94" y2="132.08" width="0.1524" layer="91"/>
+<label x="20.32" y="132.08" size="1.778" layer="95"/>
 </segment>
 </net>
@@
 </segment>
 </net>
-<net name="N$1" class="0">
-<segment>
-<pinref part="R3" gate="G$1" pin="1"/>
-<wire x1="88.9" y1="58.42" x2="91.44" y2="58.42" width="0.1524" layer="91"/>
-<pinref part="C1" gate="G$1" pin="1"/>
-<wire x1="91.44" y1="58.42" x2="91.44" y2="55.88" width="0.1524" layer="91"/>
-<pinref part="R4" gate="G$1" pin="1"/>
-<wire x1="91.44" y1="48.26" x2="88.9" y2="48.26" width="0.1524" layer="91"/>
-<wire x1="93.98" y1="55.88" x2="91.44" y2="55.88" width="0.1524" layer="91"/>
-<wire x1="91.44" y1="55.88" x2="91.44" y2="48.26" width="0.1524" layer="91"/>
-<junction x="93.98" y="55.88"/>
-</segment>
-</net>
 <net name="OIN" class="0">
 <segment>
@@
 <wire x1="200.66" y1="182.88" x2="210.82" y2="182.88" width="0.1524" layer="91"/>
 <pinref part="R10" gate="G$1" pin="1"/>
+<wire x1="200.66" y1="182.88" x2="195.58" y2="182.88" width="0.1524" layer="91"/>
+<junction x="200.66" y="182.88"/>
+<label x="195.58" y="180.34" size="1.778" layer="95"/>
 </segment>
 <segment>
@@
 <wire x1="66.04" y1="127" x2="71.12" y2="127" width="0.1524" layer="91"/>
 <label x="71.12" y="127" size="1.778" layer="95"/>
-</segment>
-<segment>
-<pinref part="Y1" gate="G$1" pin="OUT/IN"/>
-<pinref part="R10" gate="G$1" pin="2"/>
-<wire x1="200.66" y1="195.58" x2="200.66" y2="193.04" width="0.1524" layer="91"/>
-<label x="203.2" y="195.58" size="1.778" layer="95"/>
 </segment>
 </net>
@@
 </segment>
 </net>
+<net name="N$2" class="0">
+<segment>
+<pinref part="R10" gate="G$1" pin="2"/>
+<pinref part="Y1" gate="G$1" pin="OUT/IN"/>
+<wire x1="200.66" y1="193.04" x2="200.66" y2="195.58" width="0.1524" layer="91"/>
+</segment>
+</net>
+<net name="N$6" class="0">
+<segment>
+<pinref part="R4" gate="G$1" pin="1"/>
+<wire x1="91.44" y1="48.26" x2="88.9" y2="48.26" width="0.1524" layer="91"/>
+<pinref part="R3" gate="G$1" pin="1"/>
+<wire x1="88.9" y1="58.42" x2="91.44" y2="58.42" width="0.1524" layer="91"/>
+<wire x1="91.44" y1="58.42" x2="91.44" y2="55.88" width="0.1524" layer="91"/>
+<pinref part="C1" gate="G$1" pin="1"/>
+<wire x1="91.44" y1="55.88" x2="93.98" y2="55.88" width="0.1524" layer="91"/>
+<wire x1="91.44" y1="48.26" x2="91.44" y2="55.88" width="0.1524" layer="91"/>
+<junction x="91.44" y="55.88"/>
+</segment>
+</net>
 </nets>
 </sheet>
 </sheets>
+<errors>
+</errors>
 </schematic>
 </drawing>

Commit message: README
Parts:
- removed FB!: 600 uH, adafruit:R-US_R0805
- added FB1: 600 uH, adafruit:R-US_R0805
- added R11: 0, adafruit:R-US_R0805
- added R12, R8: 4.7K, adafruit:R-US_R0805
- C9: value 100nF -> 18pF
- R10: value 0 -> 4.7K; CRCW060350R0FKEA (none) -> 50
Connections:
- net TPIN+ renamed TPIN_P
- net TPIN- renamed TPIN_N
- net TPOUT+ renamed TPOUT_P
- net TPOUT- renamed TPOUT_N
- new net N$1: C2.1, FB1.2, J7.CT, R5.1, R6.1
- net 3.3V: now also FB1.1, R10.1, R12.1, R8.1; no longer C2.1, FB!.1, FB!.2, J7.CT, R5.1, R6.1
- net N$2: now also C8.1, R11.1; no longer R10.2
- net N$4: now also R8.2
- net OOUT: now also R11.2; no longer C8.1, R10.1
- net SCK: now also R10.2
- net SDA: now also R12.2
Other:
- moved on the sheet: C2, R10

Commit message: README
Parts:
- removed R11: 0, adafruit:R-US_R0805
Connections:
- removed net N$2: C8.1, R11.1, Y1.OUT/IN
- net OOUT: now also C8.1, Y1.OUT/IN; no longer R11.2
Changed lines of the file:
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@@
 <clearance class="3" value="0.254"/>
+</class>
+<class number="4" name="supply" width="0.3302" drill="0">
 </class>
 </classes>
@@
 </part>
 <part name="SYMBOL14" library="APU_ENGR480_UPS_EAGLE_Library" deviceset="3.3V" device=""/>
-<part name="R11" library="adafruit" library_urn="urn:adsk.eagle:library:420" deviceset="R-US_" device="R0805" package3d_urn="urn:adsk.eagle:package:6240566/1" value="0"/>
 <part name="R10" library="adafruit" library_urn="urn:adsk.eagle:library:420" deviceset="R-US_" device="R0805" package3d_urn="urn:adsk.eagle:package:6240566/1" value="4.7K">
 <attribute name="CRCW060350R0FKEA" value="50"/>
@@
 <attribute name="VALUE" x="109.855" y="188.595" size="1.778" layer="96"/>
 </instance>
-<instance part="R11" gate="G$1" x="193.04" y="182.88" smashed="yes" rot="R180">
-<attribute name="NAME" x="191.77" y="186.4614" size="1.778" layer="95" rot="R180"/>
-<attribute name="VALUE" x="189.23" y="181.102" size="1.778" layer="96" rot="R180"/>
-</instance>
 <instance part="R10" gate="G$1" x="170.18" y="190.5" smashed="yes" rot="R270">
 <attribute name="NAME" x="171.6786" y="194.31" size="1.778" layer="95" rot="R270"/>
@@
 </segment>
 </net>
-<net name="3.3V" class="0">
+<net name="3.3V" class="4">
 <segment>
 <pinref part="U6" gate="G$1" pin="VDDOSC"/>
@@
 </segment>
 <segment>
-<pinref part="R11" gate="G$1" pin="2"/>
-<wire x1="187.96" y1="182.88" x2="182.88" y2="182.88" width="0.1524" layer="91"/>
-<label x="180.34" y="182.88" size="1.778" layer="95"/>
+<label x="190.5" y="182.88" size="1.778" layer="95"/>
+<pinref part="C8" gate="G$1" pin="1"/>
+<wire x1="210.82" y1="182.88" x2="200.66" y2="182.88" width="0.1524" layer="91"/>
+<pinref part="Y1" gate="G$1" pin="OUT/IN"/>
+<wire x1="200.66" y1="195.58" x2="200.66" y2="182.88" width="0.1524" layer="91"/>
+<junction x="200.66" y="182.88"/>
+<wire x1="193.04" y1="182.88" x2="200.66" y2="182.88" width="0.1524" layer="91"/>
 </segment>
 </net>
@@
 </segment>
 </net>
-<net name="N$2" class="0">
-<segment>
-<pinref part="C8" gate="G$1" pin="1"/>
-<wire x1="210.82" y1="182.88" x2="200.66" y2="182.88" width="0.1524" layer="91"/>
-<pinref part="R11" gate="G$1" pin="1"/>
-<pinref part="Y1" gate="G$1" pin="OUT/IN"/>
-<wire x1="200.66" y1="182.88" x2="198.12" y2="182.88" width="0.1524" layer="91"/>
-<wire x1="200.66" y1="195.58" x2="200.66" y2="182.88" width="0.1524" layer="91"/>
-<junction x="200.66" y="182.88"/>
-</segment>
-</net>
